File: pcb/pcb.kicad_sch (KiCad schematic)
At the start: 41 parts, among them J1 NMJ4HCD2, J2 NMJ4HCD2, J3 694106301002, SW1 FSWITCH, U1 RC4558, U2 L78L09_TO92

Commit message: Finalize pcb
Connections:
- net GND: now also RV1.1, RV3.1; no longer RV1.3, RV3.3
- net at R14.2: now also RV3.3; no longer RV3.1
Other:
- note removed: "TODO: power supply barrel jack"
Changed lines of the file:
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@@
 	(generator_version "9.0")
 	(paper "A4")
-	(text "TODO: power supply barrel jack"
-		(exclude_from_sim yes)
-		(at 88.9 165.1 0)
-		(effects
-			(font
-				(size 1.27 1.27)
-			)
-		)
-	)
 	(junction
 		(at 177.8 127)
@@
 		(lib_id "Device:R_Potentiometer")
 		(at 78.74 80.01 0)
-		(mirror x)
 		(unit 1)
 		(exclude_from_sim no)
@@
 		(lib_id "Device:R_Potentiometer")
 		(at 254 146.05 0)
+		(mirror x)
 		(unit 1)
 		(exclude_from_sim no)
@@
 		(dnp no)
 		(property "Reference" "RV3"
-			(at 261.62 139.7 0)
+			(at 261.62 152.4 0)
 			(effects
 				(font
@@
 		)
 		(property "Value" "100k"
-			(at 261.62 142.24 0)
+			(at 261.62 149.86 0)
 			(effects
 				(font

Commit message: 1590b pcb
Parts:
- J1, J2: footprint NMJ4HCD2:NMJ4HCD2 -> Connector_PinHeader_2.00mm:PinHeader_1x04_P2.00mm_Vertical
- J3: footprint PowerJackFemale:694106301002 -> Connector_PinHeader_2.00mm:PinHeader_1x03_P2.00mm_Vertical
- RV1, RV2, RV3: footprint Potentiometer_THT:Potentiometer_Omeg_PC16BU_Vertical -> Connector_PinHeader_2.00mm:PinHeader_1x03_P2.00mm_Vertical
Connections:
- net GND: now also RV1.3, RV2.1
Changed lines of the file:
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@@
 			)
 		)
-		(property "Footprint" "NMJ4HCD2:NMJ4HCD2"
+		(property "Footprint" "Connector_PinHeader_2.00mm:PinHeader_1x04_P2.00mm_Vertical"
 			(at 24.13 211.76 0)
 			(effects
@@
 			)
 		)
-		(property "Footprint" "PowerJackFemale:694106301002"
+		(property "Footprint" "Connector_PinHeader_2.00mm:PinHeader_1x03_P2.00mm_Vertical"
 			(at 46.99 122.86 0)
 			(effects
@@
 			)
 		)
-		(property "Footprint" "NMJ4HCD2:NMJ4HCD2"
+		(property "Footprint" "Connector_PinHeader_2.00mm:PinHeader_1x04_P2.00mm_Vertical"
 			(at 24.13 163.5 0)
 			(effects
@@
 			)
 		)
-		(property "Footprint" "Potentiometer_THT:Potentiometer_Omeg_PC16BU_Vertical"
+		(property "Footprint" "Connector_PinHeader_2.00mm:PinHeader_1x03_P2.00mm_Vertical"
 			(at 78.74 80.01 0)
 			(effects
@@
 	)
 	(symbol
+		(lib_id "power:GND")
+		(at 78.74 83.82 0)
+		(unit 1)
+		(exclude_from_sim no)
+		(in_bom yes)
+		(on_board yes)
+		(dnp no)
+		(fields_autoplaced yes)
+		(property "Reference" "#PWR08"
+			(at 78.74 90.17 0)
+			(effects
+				(font
+					(size 1.27 1.27)
+				)
+				(hide yes)
+			)
+		)
+		(property "Value" "GND"
+			(at 78.74 88.9 0)
+			(effects
+				(font
+					(size 1.27 1.27)
+				)
+			)
+		)
+		(property "Footprint" ""
+			(at 78.74 83.82 0)
+			(effects
+				(font
+					(size 1.27 1.27)
+				)
+				(hide yes)
+			)
+		)
+		(property "Datasheet" ""
+			(at 78.74 83.82 0)
+			(effects
+				(font
+					(size 1.27 1.27)
+				)
+				(hide yes)
+			)
+		)
+		(property "Description" "Power symbol creates a global label with name \"GND\" , ground"
+			(at 78.74 83.82 0)
+			(effects
+				(font
+					(size 1.27 1.27)
+				)
+				(hide yes)
+			)
+		)
+		(pin "1"
+		)
+		(instances
+			(project "pcb"
+				(path "/0709eb16-b1b4-4efb-9d5a-efabba183f02"
+					(reference "#PWR08")
+					(unit 1)
+				)
+			)
+		)
+	)
+	(symbol
 		(lib_id "Device:C")
 		(at 107.95 76.2 90)
@@
 			)
 		)
-		(property "Footprint" "Potentiometer_THT:Potentiometer_Omeg_PC16BU_Vertical"
+		(property "Footprint" "Connector_PinHeader_2.00mm:PinHeader_1x03_P2.00mm_Vertical"
 			(at 222.25 85.09 0)
 			(effects
@@
 			)
 		)
-		(property "Footprint" "Potentiometer_THT:Potentiometer_Omeg_PC16BU_Vertical"
+		(property "Footprint" "Connector_PinHeader_2.00mm:PinHeader_1x03_P2.00mm_Vertical"
 			(at 254 146.05 0)
 			(effects
@@
 					(unit 1)
 				)
+			)
+		)
+	)
+	(symbol
+		(lib_id "power:GND")
+		(at 226.06 85.09 90)
+		(unit 1)
+		(exclude_from_sim no)
+		(in_bom yes)
+		(on_board yes)
+		(dnp no)
+		(fields_autoplaced yes)
+		(property "Reference" "#PWR016"
+			(at 232.41 85.09 0)
+			(effects
+				(font
+					(size 1.27 1.27)
+				)
+				(hide yes)
+			)
+		)
+		(property "Value" "GND"
+			(at 229.87 85.0899 90)
+			(effects
+				(font
+					(size 1.27 1.27)
+				)
+				(justify right)
+			)
+		)
+		(property "Footprint" ""
+			(at 226.06 85.09 0)
+			(effects
+				(font
+					(size 1.27 1.27)
+				)
+				(hide yes)
+			)
+		)
+		(property "Datasheet" ""
+			(at 226.06 85.09 0)
+			(effects
+				(font
+					(size 1.27 1.27)
+				)
+				(hide yes)
+			)
+		)
+		(property "Description" "Power symbol creates a global label with name \"GND\" , ground"
+			(at 226.06 85.09 0)
+			(effects
+				(font
+					(size 1.27 1.27)
+				)
+				(hide yes)
+			)
+		)
+		(pin "1"
+		)
+		(instances
+			(project "pcb"
+				(path "/0709eb16-b1b4-4efb-9d5a-efabba183f02"
+					(reference "#PWR016")
+					(unit 1)
+				)
