File: pcb/pcb.kicad_pcb (KiCad board)
At the start: 2 copper layers, 100 x 100 mm, 41 parts, among them J1 NMJ4HCD2, J2 NMJ4HCD2, J3 694106301002, SW1 FSWITCH, U1 RC4558, U2 L78L09_TO92

Commit message: Fix reverse polarity protection diode - schematic
Connections:
- C1 pad 1: /VCC -> /V9
- C14 pad 2: /VCC -> /V9
- C2 pad 1: /VCC -> /V9
- D1 pad 1: /VCC -> /VCCRAW
- J3 pad 1: /VCCRAW -> Net-(J3-POWER)
- R1 pad 2: /V9 -> Net-(J3-POWER)
- R2 pad 1: /VCC -> /V9
- SW1 pad 4: /VCC -> /V9
- U1 pad 8: /VCC -> /V9
Routing:
- net /VCC: track 79.7 -> 0.00 mm
- net (no net): track 0.00 -> 79.7 mm
Changed lines of the file:
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@@
 	(net 16 "/AMP2-")
 	(net 17 "Net-(C13-Pad2)")
-	(net 18 "/VCC")
+	(net 18 "Net-(J3-POWER)")
 	(net 19 "/VAMPIN")
 	(net 20 "/VVOLOUT")
@@
 			(layers "*.Cu" "*.Mask")
 			(remove_unused_layers no)
-			(net 18 "/VCC")
+			(net 27 "/V9")
 			(pintype "passive")
 		)
@@
 			(layers "*.Cu" "*.Mask")
 			(remove_unused_layers no)
-			(net 18 "/VCC")
+			(net 27 "/V9")
 			(pintype "passive")
 		)
@@
 			(layers "*.Cu" "*.Mask")
 			(remove_unused_layers no)
-			(net 18 "/VCC")
+			(net 27 "/V9")
 			(pintype "passive")
 		)
@@
 			(layers "*.Cu" "*.Mask")
 			(remove_unused_layers no)
-			(net 27 "/V9")
+			(net 18 "Net-(J3-POWER)")
 			(pintype "passive")
 		)
@@
 			(layers "*.Cu" "*.Mask")
 			(remove_unused_layers no)
-			(net 4 "/VCCRAW")
+			(net 18 "Net-(J3-POWER)")
 			(pinfunction "POWER")
 			(pintype "passive")
@@
 			(layers "*.Cu" "*.Mask")
 			(remove_unused_layers no)
-			(net 18 "/VCC")
+			(net 27 "/V9")
 			(pinfunction "V+")
 			(pintype "power_in")
@@
 			(remove_unused_layers no)
 			(roundrect_rratio 0.15625)
-			(net 18 "/VCC")
+			(net 4 "/VCCRAW")
 			(pinfunction "K")
 			(pintype "passive")
@@
 			(remove_unused_layers no)
 			(roundrect_rratio 0.1968503937)
-			(net 18 "/VCC")
+			(net 27 "/V9")
 			(pinfunction "4")
 			(pintype "bidirectional")
@@
 			(layers "*.Cu" "*.Mask")
 			(remove_unused_layers no)
-			(net 18 "/VCC")
+			(net 27 "/V9")
 			(pintype "passive")
 		)
@@
 	)
 	(segment
+		(start 153.81 80.87)
+		(end 153.81 80.19)
+		(width 0.2)
+		(layer "F.Cu")
+		(net 0)
+	)
+	(segment
+		(start 159.35 79.1)
+		(end 159.45 79)
+		(width 0.2)
+		(layer "F.Cu")
+		(net 0)
+	)
+	(segment
+		(start 154.9 79.1)
+		(end 159.35 79.1)
+		(width 0.2)
+		(layer "F.Cu")
+		(net 0)
+	)
+	(segment
+		(start 163.3 83.8)
+		(end 163.3 86.2)
+		(width 0.5)
+		(layer "F.Cu")
+		(net 0)
+	)
+	(segment
+		(start 175.28 96.33)
+		(end 175.28 96.1)
+		(width 0.5)
+		(layer "F.Cu")
+		(net 0)
+	)
+	(segment
+		(start 178.05 101.75)
+		(end 180.7 101.75)
+		(width 0.5)
+		(layer "F.Cu")
+		(net 0)
+	)
+	(segment
+		(start 163.3 86.2)
+		(end 173.2 96.1)
+		(width 0.5)
+		(layer "F.Cu")
+		(net 0)
+	)
+	(segment
+		(start 169.6 105.4)
+		(end 162.9 105.4)
+		(width 0.5)
+		(layer "F.Cu")
+		(net 0)
+	)
+	(segment
+		(start 178.05 101.75)
+		(end 177.55 102.25)
+		(width 0.5)
+		(layer "F.Cu")
+		(net 0)
+	)
+	(segment
+		(start 172.75 102.25)
+		(end 169.6 105.4)
+		(width 0.5)
+		(layer "F.Cu")
+		(net 0)
+	)
+	(segment
+		(start 156.7 111.6)
+		(end 152.6 111.6)
+		(width 0.5)
+		(layer "F.Cu")
+		(net 0)
+	)
+	(segment
+		(start 180.7 101.75)
+		(end 175.28 96.33)
+		(width 0.5)
+		(layer "F.Cu")
+		(net 0)
+	)
+	(segment
+		(start 160.9 81.4)
+		(end 154.34 81.4)
+		(width 0.5)
+		(layer "F.Cu")
+		(net 0)
+	)
+	(segment
+		(start 173.2 96.1)
+		(end 175.28 96.1)
+		(width 0.5)
+		(layer "F.Cu")
+		(net 0)
+	)
+	(segment
+		(start 177.55 102.25)
+		(end 173.6 102.25)
+		(width 0.5)
+		(layer "F.Cu")
+		(net 0)
+	)
+	(segment
+		(start 152.6 111.6)
+		(end 150.2 114)
+		(width 0.5)
+		(layer "F.Cu")
+		(net 0)
+	)
+	(segment
+		(start 150.2 114)
+		(end 150 114)
+		(width 0.5)
+		(layer "F.Cu")
+		(net 0)
+	)
+	(segment
+		(start 162.9 105.4)
+		(end 156.7 111.6)
+		(width 0.5)
+		(layer "F.Cu")
+		(net 0)
+	)
+	(segment
+		(start 153.81 80.19)
+		(end 154.9 79.1)
+		(width 0.2)
+		(layer "F.Cu")
+		(net 0)
+	)
+	(segment
+		(start 173.6 102.25)
+		(end 172.75 102.25)
+		(width 0.5)
+		(layer "F.Cu")
+		(net 0)
+	)
+	(segment
+		(start 163.3 83.8)
+		(end 160.9 81.4)
+		(width 0.5)
+		(layer "F.Cu")
+		(net 0)
+	)
+	(segment
+		(start 154.34 81.4)
+		(end 153.81 80.87)
+		(width 0.5)
+		(layer "F.Cu")
+		(net 0)
+	)
+	(segment
 		(start 158.4 93.96)
 		(end 158.4 95.9)
@@
 	)
 	(segment
-		(start 153.81 80.87)
-		(end 153.81 80.19)
-		(width 0.2)
-		(layer "F.Cu")
-		(net 18)
-	)
-	(segment
-		(start 159.35 79.1)
-		(end 159.45 79)
-		(width 0.2)
-		(layer "F.Cu")
-		(net 18)
-	)
-	(segment
-		(start 154.9 79.1)
-		(end 159.35 79.1)
-		(width 0.2)
-		(layer "F.Cu")
-		(net 18)
-	)
-	(segment
-		(start 163.3 83.8)
-		(end 163.3 86.2)
-		(width 0.5)
-		(layer "F.Cu")
-		(net 18)
-	)
-	(segment
-		(start 175.28 96.33)
-		(end 175.28 96.1)
-		(width 0.5)
-		(layer "F.Cu")
-		(net 18)
-	)
-	(segment
-		(start 178.05 101.75)
-		(end 180.7 101.75)
-		(width 0.5)
-		(layer "F.Cu")
-		(net 18)
-	)
-	(segment
-		(start 163.3 86.2)
-		(end 173.2 96.1)
-		(width 0.5)
-		(layer "F.Cu")
-		(net 18)
-	)
-	(segment
-		(start 169.6 105.4)
-		(end 162.9 105.4)
-		(width 0.5)
-		(layer "F.Cu")
-		(net 18)
-	)
-	(segment
-		(start 178.05 101.75)
-		(end 177.55 102.25)
-		(width 0.5)
-		(layer "F.Cu")
-		(net 18)
-	)
-	(segment
-		(start 172.75 102.25)
-		(end 169.6 105.4)
-		(width 0.5)
-		(layer "F.Cu")
-		(net 18)
-	)
-	(segment
-		(start 156.7 111.6)
-		(end 152.6 111.6)
-		(width 0.5)
-		(layer "F.Cu")
-		(net 18)
-	)
-	(segment
-		(start 180.7 101.75)
-		(end 175.28 96.33)
-		(width 0.5)
-		(layer "F.Cu")
-		(net 18)
-	)
-	(segment
-		(start 160.9 81.4)
-		(end 154.34 81.4)
-		(width 0.5)
-		(layer "F.Cu")
-		(net 18)
-	)
-	(segment
-		(start 173.2 96.1)
-		(end 175.28 96.1)
-		(width 0.5)
-		(layer "F.Cu")
-		(net 18)
-	)
-	(segment
-		(start 177.55 102.25)
-		(end 173.6 102.25)
-		(width 0.5)
-		(layer "F.Cu")
-		(net 18)
-	)
-	(segment
-		(start 152.6 111.6)
-		(end 150.2 114)
-		(width 0.5)
-		(layer "F.Cu")
-		(net 18)
-	)
-	(segment
-		(start 150.2 114)
-		(end 150 114)
-		(width 0.5)
-		(layer "F.Cu")
-		(net 18)
-	)
-	(segment
-		(start 162.9 105.4)
-		(end 156.7 111.6)
-		(width 0.5)
-		(layer "F.Cu")
-		(net 18)
-	)
-	(segment
-		(start 153.81 80.19)
-		(end 154.9 79.1)
-		(width 0.2)
-		(layer "F.Cu")
-		(net 18)
-	)
-	(segment
-		(start 173.6 102.25)
-		(end 172.75 102.25)
-		(width 0.5)
-		(layer "F.Cu")
-		(net 18)
-	)
-	(segment
-		(start 163.3 83.8)
-		(end 160.9 81.4)
-		(width 0.5)
-		(layer "F.Cu")
-		(net 18)
-	)
-	(segment
-		(start 154.34 81.4)
-		(end 153.81 80.87)
-		(width 0.5)
-		(layer "F.Cu")
-		(net 18)
-	)
-	(segment
